File: control-module/For Micro/control-module.kicad_pcb (KiCad board)
At the start: 2 copper layers, 63.5 x 68.1 mm, 40 parts, among them J1 For Expansion, J2 For Light Sensor, J3 From Solar Panel, J4 To Flow Module (F), J5 For Flow Module b, J6 For Flow Module a, Q1 NMOS, Q2 NMOS, Q3 NMOS, Q4 NMOS, U1 TR_SERIES, U2 TR_SERIES, U3 ARDUINO_MICRO_SHIELD

Commit message: PCB Design update
Parts:
- removed I2Crepeater1, I2Crepeater2: I2C-PCA9517, Housings_SSOP:TSSOP-8_3x3mm_Pitch0.65mm
- removed J6: For Flow Module a, valveteam-footprints:Molex_KK-6410-06_06x2.54mm_Straight
- removed Q1, Q2, Q3, Q4: NMOS, TO_SOT_Packages_SMD:SOT-23_Handsoldering
- removed R1, R2: 4.7k, Resistors_SMD:R_0805_HandSoldering
- removed REF** (x3): MountingHole_2.2mm_M2, Mounting_Holes:MountingHole_2.2mm_M2
Connections:
- J1 pad 3: SDAC -> MOSI
- J1 pad 4: SCLC -> MISO
- J2 pad 2: INT -> (no net)
- J2 pad 5: DVI -> (no net)
- U3 pad 2: SDAB -> SDAA
- U3 pad 3: SCLB -> SCLA
- U3 pad 3.3V: Net-(U3-Pad3.3V) -> (no net)
- U3 pad 4: EN1/M -> (no net)
- U3 pad 6: INT/M -> (no net)
- U3 pad 7: DVI/M -> (no net)
- U3 pad A2: EN2/M -> (no net)
- U3 pad A4: Net-(U3-PadA4) -> (no net)
- U3 pad A5: Net-(U3-PadA5) -> (no net)
- U3 pad MI: Net-(U3-PadMI) -> (no net)
- U3 pad MO: Net-(U3-PadMO) -> MOSI
- U3 pad RX: Net-(U3-PadRX) -> (no net)
- U3 pad SCK: Net-(U3-PadSCK) -> MISO
- U3 pad SS: Net-(U3-PadSS) -> (no net)
- U3 pad TX: Net-(U3-PadTX) -> (no net)
Routing:
- net (no net): track 0.11 -> 216.6 mm, vias 0 -> 12
- net MISO: track 0.00 -> 97.3 mm
- net MOSI: track 0.00 -> 85.1 mm
- net SDAC: track 84.9 -> 0.00 mm
- net SCLC: track 80.2 -> 0.00 mm
- net EN2: track 74.8 -> 0.00 mm, vias 2 -> 0
- net GND: track 184.2 -> 113.3 mm, vias 17 -> 12
- net EN1: track 57.3 -> 0.00 mm, vias 4 -> 0
- net SDAB: track 53.5 -> 0.00 mm, vias 2 -> 0
- net SCLA: track 27.0 -> 76.7 mm, vias 0 -> 5
- net SCLB: track 47.8 -> 0.00 mm, vias 4 -> 0
- net EN1/M: track 47.3 -> 0.00 mm, vias 2 -> 0
- net SDAA: track 26.8 -> 70.9 mm, vias 1 -> 4
- net DVI/M: track 37.9 -> 0.00 mm, vias 4 -> 0
- net INT: track 36.8 -> 0.00 mm, vias 2 -> 0
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