File: control-module/For Micro/control-module.sch (KiCad schematic (older format))
At the start: 37 parts, among them J1 For Expansion, J2 For Light Sensor, J3 From Solar Panel, J4 To Flow Module (F), J5 For Flow Module b, J6 For Flow Module a, Q1 NMOS, Q2 NMOS, Q3 NMOS, Q4 NMOS, U1 TR_SERIES, U2 TR_SERIES, U3 ARDUINO_MICRO_SHIELD

Commit message: PCB Design update
Parts:
- removed I2Crepeater1, I2Crepeater2: I2C-PCA9517, Housings_SSOP:TSSOP-8_3x3mm_Pitch0.65mm, symbol I2C-PCA9517
- removed J6: For Flow Module a, valveteam-footprints:Molex_KK-6410-06_06x2.54mm_Straight, symbol Conn_01x06
- removed Q1, Q2, Q3, Q4: NMOS, TO_SOT_Packages_SMD:SOT-23_Handsoldering, symbol Q_NMOS_DGS
- removed R1, R2: 4.7k, Resistors_SMD:R_0805_HandSoldering, symbol R
Connections:
- net SCLB is gone; now on net SCLA: U3.3 (3(PWM)/SCL)
- net SCLC is gone; now on net MISO: J1.4 (Pin_4)
- net SDAB is gone; now on net SDAA: U3.2 (2/SDA)
- net SDAC is gone; now on net MOSI: J1.3 (Pin_3)
- net MOSI: now reaches U3.MO (MOSI)
- net MISO: now reaches U3.SCK
- net DVI/M: no longer names the net of U3.7
- net EN1/M: no longer names the net of U3.4 (4/A6)
- net EN2/M: no longer names the net of U3.A2
- net INT/M: no longer names the net of U3.6 (6(PWM)/A7)
Other:
- note removed: "I2C Pullup Resistors"
- note removed: "MOSFET Pull Down Circuits (E)\n"
