File: flow-module/flow-module.sch (KiCad schematic (older format))
At the start: 19 parts, among them P1 TERM_01X02, P2 MOLEX_01X06, P3 MOLEX_01X06, P4 TERM_01X02, P5 TERM_01X02

Commit message: PCB Design update
Parts:
- removed D1, D2, D3, D4: D, ValveTeam:do219ab, symbol D
- removed D7: LED, LEDs:LED_0805_HandSoldering, symbol LED
- removed H1: L298P, ValveTeam:powerso-20, symbol L298P
- removed P2: MOLEX_01X06, ValveTeam:Molex_KK-6410-06_06x2.54mm_Straight, symbol CONN_01X06
- removed P4: TERM_01X02, ValveTeam:TE_TERM, symbol CONN_01X02
- removed R3: 330, Resistors_SMD:R_0805_HandSoldering, symbol R
Connections:
- no-connect marks 11 -> 0

Commit message: saved changes.
Parts:
- C1, C2: symbol C -> Device:C
- D5, D6: symbol LED -> flow-module-rescue:LED
- H2: symbol LMD18201T -> flow-module-rescue:LMD18201T
- P1, P5: symbol CONN_01X02 -> flow-module-rescue:CONN_01X02
- P3: symbol CONN_01X06 -> flow-module-rescue:CONN_01X06
- R1, R2: symbol R -> Device:R
Changed lines of the file:
@@
-EESchema Schematic File Version 2
-LIBS:power
-LIBS:device
-LIBS:transistors
-LIBS:conn
-LIBS:linear
-LIBS:regul
-LIBS:74xx
-LIBS:cmos4000
-LIBS:adc-dac
-LIBS:memory
-LIBS:xilinx
-LIBS:microcontrollers
-LIBS:dsp
-LIBS:microchip
-LIBS:analog_switches
-LIBS:motorola
-LIBS:texas
-LIBS:intel
-LIBS:audio
-LIBS:interface
-LIBS:digital-audio
-LIBS:philips
-LIBS:display
-LIBS:cypress
-LIBS:siliconi
-LIBS:opto
-LIBS:atmel
-LIBS:contrib
-LIBS:valves
-LIBS:valveteam
+EESchema Schematic File Version 4
 LIBS:flow-module-cache
-EELAYER 25 0
+EELAYER 26 0
 EELAYER END
 $Descr A4 11693 8268
@@
 $EndDescr
 $Comp
-L CONN_01X06 P3
+L flow-module-rescue:CONN_01X06 P3
 U 1 1 5B04304C
 P 1000 3000
@@
 $EndComp
 $Comp
-L CONN_01X02 P5
+L flow-module-rescue:CONN_01X02 P5
 U 1 1 5B043210
 P 5650 3100
@@
 $EndComp
 $Comp
-L CONN_01X02 P1
+L flow-module-rescue:CONN_01X02 P1
 U 1 1 5B0432BB
 P 950 850
@@
 $EndComp
 $Comp
-L Earth #PWR01
+L power:Earth #PWR01
 U 1 1 5B043C8F
 P 1150 900
@@
 $EndComp
 $Comp
-L VCC #PWR02
+L power:VCC #PWR02
 U 1 1 5B043F32
 P 1150 800
@@
 From Power Supply
 $Comp
-L VAA #PWR03
+L power:VAA #PWR03
 U 1 1 5B045A4D
 P 1200 3250
@@
 $EndComp
 $Comp
-L Earth #PWR04
+L power:Earth #PWR04
 U 1 1 5B045A74
 P 1200 2750
@@
 $EndComp
 $Comp
-L LMD18201T H2
+L flow-module-rescue:LMD18201T H2
 U 1 1 5B043BC1
 P 3250 2900
@@
 Connection ~ 3700 2950
 $Comp
-L Earth #PWR05
+L power:Earth #PWR05
 U 1 1 5B043D56
 P 3850 2950
@@
 Output1
 $Comp
-L VCC #PWR06
+L power:VCC #PWR06
 U 1 1 5B0448D2
 P 3700 3150
@@
 $EndComp
 Wire Wire Line
-	3700 2750 4100 2750
-Wire Wire Line
-	3700 3550 4100 3550
-$Comp
-L C C1
+	3700 2750 4000 2750
+Wire Wire Line
+	3700 3550 4000 3550
+$Comp
+L Device:C C1
 U 1 1 5B045DA5
 P 3850 2650
@@
 Connection ~ 4000 2750
 $Comp
-L C C2
+L Device:C C2
 U 1 1 5B0461EC
 P 3850 3650
@@
 From Control Module\n
 $Comp
-L VCC #PWR07
+L power:VCC #PWR07
 U 1 1 5B052ACC
 P 6450 1150
@@
 $EndComp
 $Comp
-L VAA #PWR08
+L power:VAA #PWR08
 U 1 1 5B052B8B
 P 6800 1150
@@
 $EndComp
 $Comp
-L LED D5
+L flow-module-rescue:LED D5
 U 1 1 5B052BE4
 P 6450 1350
@@
 $EndComp
 $Comp
-L LED D6
+L flow-module-rescue:LED D6
 U 1 1 5B052C8D
 P 6800 1350
@@
 $EndComp
 $Comp
-L R R1
+L Device:R R1
 U 1 1 5B052D3E
 P 6450 1700
@@
 $EndComp
 $Comp
-L R R2
+L Device:R R2
 U 1 1 5B052DC4
 P 6800 1700
@@
 $EndComp
 $Comp
-L Earth #PWR09
+L power:Earth #PWR09
 U 1 1 5B052E71
 P 6450 1850
@@
 $EndComp
 $Comp
-L Earth #PWR010
+L power:Earth #PWR010
 U 1 1 5B052EB5
 P 6800 1850
@@
 Text Notes 6450 2100 0    60   ~ 0
 Status LEDs\n
+Wire Wire Line
+	4000 2750 4100 2750
+Wire Wire Line
+	4000 3550 4100 3550
 $EndSCHEMATC
